Commit message: Refactor project structure and update configurations for SLAM integration
- Removed deprecated Python hook scripts for rescue_raspberry_brain and rescue_pc_brain.
- Updated local setup scripts to reflect new installation paths.
- Modified package.xml files to remove unnecessary dependencies.
- Adjusted slam_toolbox parameters in slam.launch.py for improved functionality.
- Added Dockerfile for containerized environment setup with necessary dependencies.
- Created run_slam_container.sh script for simplified container management and SLAM execution.
- Introduced udev rules for hardware device permissions.
- Updated robot description URDF to remove unnecessary properties.

File: src/rescue_robot_description/urdf/rescue_robot.urdf.xacro (robot description, xacro)
@@ -17,5 +17,4 @@
   <xacro:property name="lidar_height"     value="0.04"/>   <!-- alto lidar [m] -->
   <xacro:property name="lidar_z_offset"   value="0.10"/>   <!-- altura desde tope de cuerpo [m] -->
-  <xacro:property name="pi" value="3.14159265358979"/>
   <!-- ── Materiales ── -->
   <material name="dark_gray"><color rgba="0.2 0.2 0.2 1.0"/></material>

Commit message: Add point cloud accumulation publisher and update RViz configuration

File: src/rescue_robot_description/urdf/rescue_robot.urdf.xacro (robot description, xacro)
@@ -169,5 +169,6 @@
     <parent link="base_link"/>
     <child  link="camera_link"/>
-    <origin xyz="${base_length/2 - 0.01} 0 ${base_height/2 + 0.05}"
+    <!-- Cara delantera: x = base_length/2 + mitad caja cámara, altura original -->
+    <origin xyz="${base_length/2 + 0.02} 0 ${base_height/2 + 0.05}"
             rpy="0 0.261 0"/>  <!-- 15° pitch down = 0.261 rad -->
   </joint>
